File: hardware/midi_euro.kicad_sch (KiCad schematic)
At the start: 0 parts

Commit message: chore: resync local state
Other:
- sheet IOs renamed pitch
- added sheet Gates (gates.kicad_sch)
- added sheet velocity (velocity.kicad_sch)
